File: eagle/Theremin/Theremin.brd (EAGLE design)
At the start: 254 x 101.6 mm, 0 parts

Commit message: Theremin board design
Parts:
- added C16: 22pF, SparkFun-Passives:CAP-PTH-SMALLEZ
- added C17, C18: 1uF, SparkFun-Passives:CPOL-RADIAL-10UF-25V
- added Q6, Q7, Q8: 2N3904, transistor:TO92
- added R15, R17, R19: 470, SparkFun-Passives:AXIAL-0.3EZ
- added R16, R21: 2.2K, SparkFun-Passives:AXIAL-0.3EZ
- added R18: 2.7K, SparkFun-Passives:AXIAL-0.3EZ
- added R20: 33, SparkFun-Passives:AXIAL-0.3EZ
- added R22, R40: 10K, SparkFun-Passives:AXIAL-0.3EZ
Connections:
- new net -12V: R16.P$1, R22.P$1, R40.P$1
- new net GND: C18.1, R15.P$1, R21.P$1
- new net N$1: Q8.2, R19.P$1
- new net N$2: C16.2, R19.P$2, R20.P$2
- new net N$3: C17.1, R20.P$1, R21.P$2, R22.P$2
- new net N$4: C16.1, Q8.1
- new net N$5: C17.2, C18.2, Q8.3, R18.P$2, R40.P$2
- new net N$6: Q6.3, Q7.3, R16.P$2
- new net N$7: R18.P$1
- new net N$8: Q6.2
- new net N$9: Q7.2, R17.P$2
Changed lines of the file:
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@@
 <setting verticaltext="up"/>
 </settings>
-<grid distance="0.1" unitdist="inch" unit="inch" style="lines" multiple="1" display="yes" altdistance="0.025" altunitdist="inch" altunit="inch"/>
+<grid distance="0.05" unitdist="inch" unit="inch" style="lines" multiple="1" display="yes" altdistance="0.025" altunitdist="inch" altunit="inch"/>
 <layers>
 <layer number="1" name="Top" color="4" fill="1" visible="yes" active="yes"/>
@@
 <layer number="48" name="Document" color="7" fill="1" visible="yes" active="yes"/>
 <layer number="49" name="Reference" color="7" fill="1" visible="yes" active="yes"/>
+<layer number="50" name="dxf" color="7" fill="1" visible="no" active="no"/>
 <layer number="51" name="tDocu" color="7" fill="1" visible="yes" active="yes"/>
 <layer number="52" name="bDocu" color="7" fill="1" visible="yes" active="yes"/>
+<layer number="53" name="tGND_GNDA" color="7" fill="9" visible="no" active="no"/>
+<layer number="54" name="bGND_GNDA" color="1" fill="9" visible="no" active="no"/>
+<layer number="56" name="wert" color="7" fill="1" visible="no" active="no"/>
 <layer number="91" name="Nets" color="2" fill="1" visible="no" active="no"/>
 <layer number="92" name="Busses" color="1" fill="1" visible="no" active="no"/>
@@
 <layer number="97" name="Info" color="7" fill="1" visible="no" active="no"/>
 <layer number="98" name="Guide" color="6" fill="1" visible="no" active="no"/>
+<layer number="100" name="Muster" color="7" fill="1" visible="no" active="no"/>
+<layer number="101" name="Patch_Top" color="12" fill="4" visible="no" active="yes"/>
+<layer number="102" name="Vscore" color="7" fill="1" visible="no" active="yes"/>
+<layer number="103" name="tMap" color="7" fill="1" visible="no" active="yes"/>
+<layer number="104" name="Name" color="16" fill="1" visible="no" active="yes"/>
+<layer number="105" name="tPlate" color="7" fill="1" visible="no" active="yes"/>
+<layer number="106" name="bPlate" color="7" fill="1" visible="no" active="yes"/>
+<layer number="107" name="Crop" color="7" fill="1" visible="no" active="yes"/>
+<layer number="116" name="Patch_BOT" color="9" fill="4" visible="no" active="yes"/>
+<layer number="121" name="_tsilk" color="7" fill="1" visible="no" active="yes"/>
+<layer number="122" name="_bsilk" color="7" fill="1" visible="no" active="yes"/>
+<layer number="125" name="_tNames" color="7" fill="1" visible="no" active="yes"/>
+<layer number="144" name="Drill_legend" color="7" fill="1" visible="no" active="yes"/>
+<layer number="151" name="HeatSink" color="7" fill="1" visible="no" active="yes"/>
+<layer number="200" name="200bmp" color="1" fill="10" visible="no" active="yes"/>
+<layer number="201" name="201bmp" color="2" fill="10" visible="no" active="yes"/>
+<layer number="202" name="202bmp" color="3" fill="10" visible="no" active="yes"/>
+<layer number="203" name="203bmp" color="4" fill="10" visible="no" active="yes"/>
+<layer number="204" name="204bmp" color="5" fill="10" visible="no" active="yes"/>
+<layer number="205" name="205bmp" color="6" fill="10" visible="no" active="yes"/>
+<layer number="206" name="206bmp" color="7" fill="10" visible="no" active="yes"/>
+<layer number="207" name="207bmp" color="8" fill="10" visible="no" active="yes"/>
+<layer number="208" name="208bmp" color="9" fill="10" visible="no" active="yes"/>
+<layer number="209" name="209bmp" color="7" fill="1" visible="no" active="yes"/>
+<layer number="210" name="210bmp" color="7" fill="1" visible="no" active="yes"/>
+<layer number="211" name="211bmp" color="7" fill="1" visible="no" active="yes"/>
+<layer number="212" name="212bmp" color="7" fill="1" visible="no" active="yes"/>
+<layer number="213" name="213bmp" color="7" fill="1" visible="no" active="yes"/>
+<layer number="214" name="214bmp" color="7" fill="1" visible="no" active="yes"/>
+<layer number="215" name="215bmp" color="7" fill="1" visible="no" active="yes"/>
+<layer number="216" name="216bmp" color="7" fill="1" visible="no" active="yes"/>
+<layer number="217" name="217bmp" color="18" fill="1" visible="no" active="no"/>
+<layer number="218" name="218bmp" color="19" fill="1" visible="no" active="no"/>
+<layer number="219" name="219bmp" color="20" fill="1" visible="no" active="no"/>
+<layer number="220" name="220bmp" color="21" fill="1" visible="no" active="no"/>
+<layer number="221" name="221bmp" color="22" fill="1" visible="no" active="no"/>
+<layer number="222" name="222bmp" color="23" fill="1" visible="no" active="no"/>
+<layer number="223" name="223bmp" color="24" fill="1" visible="no" active="no"/>
+<layer number="224" name="224bmp" color="25" fill="1" visible="no" active="no"/>
+<layer number="250" name="Descript" color="3" fill="1" visible="no" active="no"/>
+<layer number="251" name="SMDround" color="12" fill="11" visible="no" active="no"/>
+<layer number="254" name="cooling" color="7" fill="1" visible="no" active="yes"/>
 </layers>
 <board>
@@
 </autorouter>
 <elements>
+<element name="Q8" library="transistor" package="TO92" value="2N3904" x="15.24" y="45.72"/>
+<element name="R19" library="SparkFun-Passives" package="AXIAL-0.3EZ" value="470" x="15.24" y="29.21"/>
+<element name="R15" library="SparkFun-Passives" package="AXIAL-0.3EZ" value="470" x="15.24" y="40.64"/>
+<element name="R17" library="SparkFun-Passives" package="AXIAL-0.3EZ" value="470" x="15.24" y="36.83"/>
+<element name="R18" library="SparkFun-Passives" package="AXIAL-0.3EZ" value="2.7K" x="15.24" y="25.4"/>
+<element name="R20" library="SparkFun-Passives" package="AXIAL-0.3EZ" value="33" x="15.24" y="33.02"/>
+<element name="C17" library="SparkFun-Passives" package="CPOL-RADIAL-10UF-25V" value="1uF" x="11.43" y="19.05" rot="R180"/>
+<element name="C18" library="SparkFun-Passives" package="CPOL-RADIAL-10UF-25V" value="1uF" x="19.05" y="19.05" rot="R180"/>
+<element name="C16" library="SparkFun-Passives" package="CAP-PTH-SMALLEZ" value="22pF" x="24.13" y="38.1" rot="R270"/>
+<element name="R22" library="SparkFun-Passives" package="AXIAL-0.3EZ" value="10K" x="34.29" y="24.13"/>
+<element name="R21" library="SparkFun-Passives" package="AXIAL-0.3EZ" value="2.2K" x="34.29" y="26.67"/>
+<element name="R40" library="SparkFun-Passives" package="AXIAL-0.3EZ" value="10K" x="34.29" y="21.59"/>
+<element name="Q7" library="transistor" package="TO92" value="2N3904" x="36.83" y="46.99" rot="R90"/>
+<element name="Q6" library="transistor" package="TO92" value="2N3904" x="30.48" y="46.99" rot="R90"/>
+<element name="R16" library="SparkFun-Passives" package="AXIAL-0.3EZ" value="2.2K" x="34.29" y="19.05"/>
 </elements>
 <signals>
+<signal name="N$1">
+<contactref element="Q8" pad="2"/>
+<contactref element="R19" pad="P$1"/>
+<wire x1="11.43" y1="29.21" x2="15.24" y2="47.625" width="0" layer="19" extent="1-1"/>
+</signal>
+<signal name="N$2">
+<contactref element="R19" pad="P$2"/>
+<contactref element="R20" pad="P$2"/>
+<contactref element="C16" pad="2"/>
+<wire x1="19.05" y1="29.21" x2="19.05" y2="33.02" width="0" layer="19" extent="1-1"/>
+<wire x1="24.13" y1="35.56" x2="19.05" y2="29.21" width="0" layer="19" extent="1-1"/>
+</signal>
+<signal name="N$3">
+<contactref element="C17" pad="1"/>
+<contactref element="R20" pad="P$1"/>
+<contactref element="R22" pad="P$2"/>
+<contactref element="R21" pad="P$2"/>
+<wire x1="10.16" y1="19.05" x2="11.43" y2="33.02" width="0" layer="19" extent="1-1"/>
+<wire x1="38.1" y1="24.13" x2="10.16" y2="19.05" width="0" layer="19" extent="1-1"/>
+<wire x1="38.1" y1="26.67" x2="38.1" y2="24.13" width="0" layer="19" extent="1-1"/>
+</signal>
+<signal name="N$4">
+<contactref element="Q8" pad="1"/>
+<contactref element="C16" pad="1"/>
+<wire x1="24.13" y1="38.1" x2="16.51" y2="45.72" width="0" layer="19" extent="1-1"/>
+</signal>
+<signal name="N$5">
+<contactref element="C17" pad="2"/>
+<contactref element="Q8" pad="3"/>
+<contactref element="R18" pad="P$2"/>
+<contactref element="C18" pad="2"/>
+<contactref element="R40" pad="P$2"/>
+<wire x1="19.05" y1="25.4" x2="13.97" y2="45.72" width="0" layer="19" extent="1-1"/>
+<wire x1="20.32" y1="19.05" x2="19.05" y2="25.4" width="0" layer="19" extent="1-1"/>
+<wire x1="12.7" y1="19.05" x2="20.32" y2="19.05" width="0" layer="19" extent="1-1"/>
+<wire x1="38.1" y1="21.59" x2="12.7" y2="19.05" width="0" layer="19" extent="1-1"/>
+</signal>
+<signal name="GND">
+<contactref element="R21" pad="P$1"/>
+<contactref element="C18" pad="1"/>
+<contactref element="R15" pad="P$1"/>
+<wire x1="17.78" y1="19.05" x2="30.48" y2="26.67" width="0" layer="19" extent="1-1"/>
+<wire x1="11.43" y1="40.64" x2="17.78" y2="19.05" width="0" layer="19" extent="1-1"/>
+</signal>
+<signal name="N$7">
+<contactref element="R18" pad="P$1"/>
+</signal>
+<signal name="-12V">
+<contactref element="R22" pad="P$1"/>
+<contactref element="R40" pad="P$1"/>
+<contactref element="R16" pad="P$1"/>
+<wire x1="30.48" y1="21.59" x2="30.48" y2="24.13" width="0" layer="19" extent="1-1"/>
+<wire x1="30.48" y1="19.05" x2="30.48" y2="21.59" width="0" layer="19" extent="1-1"/>
+</signal>
+<signal name="N$6">
+<contactref element="Q7" pad="3"/>
+<contactref element="Q6" pad="3"/>
+<contactref element="R16" pad="P$2"/>
+<wire x1="36.83" y1="45.72" x2="30.48" y2="45.72" width="0" layer="19" extent="1-1"/>
+<wire x1="38.1" y1="19.05" x2="30.48" y2="45.72" width="0" layer="19" extent="1-1"/>
+</signal>
+<signal name="N$8">
+<contactref element="Q6" pad="2"/>
+</signal>
+<signal name="N$9">
+<contactref element="Q7" pad="2"/>
+<contactref element="R17" pad="P$2"/>
+<wire x1="19.05" y1="36.83" x2="34.925" y2="46.99" width="0" layer="19" extent="1-1"/>
+</signal>
 </signals>
 </board>

Commit message: get everything committed to move to new machine
Parts:
- added C13: 22uF, SparkFun-Capacitors:CPOL-RADIAL-1000UF-25V
- added C14: 1800pF, SparkFun-Capacitors:CAP-PTH-LARGE
- added C15: 6800pF, capacitor-wima:C5B3
- added D1, D3: 1N4004, diode:DO41-10
- added L11: 47uH, marky-parts:SLOT-TEN
- added L14: 22uH, marky-parts:FIXED-INDUCTOR-API-DELEVAN
- added U1: LM78L12, marky-parts:TO-92
- added U2: LM79L12, marky-parts:TO-92
- Q6, Q7: value 2N3904 -> (none)
- moved R21 2.54 mm to (34.3, 24.1)
- moved R16 2.54 mm to (34.3, 16.5)
- moved R22 2.54 mm to (34.3, 21.6)
- moved R40 2.54 mm to (34.3, 19.1)
Connections:
- new net N$10: C13.1, L11.IN$1, Q7.1
- new net N$11: L11.OUT$3, L14.P$1
- new net N$12: D3.A, U2.2
- new net N$13: D1.C, U1.1
- net GND: now also C13.2, C15.2, L11.TAB@7, L11.TAB@8, R17.P$1, U1.2, U2.3
- net N$4: now also C14.1, L14.P$2, Q6.1
- net N$8: now also R15.P$2
- net N$9: now also C14.2, C15.1
Other:
- board text added: "VOL OSC & TUNING"
Changed lines of the file:
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@@
 <setting verticaltext="up"/>
 </settings>
-<grid distance="0.05" unitdist="inch" unit="inch" style="lines" multiple="1" display="yes" altdistance="0.025" altunitdist="inch" altunit="inch"/>
+<grid distance="0.0125" unitdist="inch" unit="inch" style="lines" multiple="1" display="yes" altdistance="0.025" altunitdist="inch" altunit="inch"/>
 <layers>
 <layer number="1" name="Top" color="4" fill="1" visible="yes" active="yes"/>
@@
 <layer number="106" name="bPlate" color="7" fill="1" visible="no" active="yes"/>
 <layer number="107" name="Crop" color="7" fill="1" visible="no" active="yes"/>
+<layer number="108" name="tplace-old" color="10" fill="1" visible="yes" active="yes"/>
+<layer number="109" name="ref-old" color="11" fill="1" visible="yes" active="yes"/>
 <layer number="116" name="Patch_BOT" color="9" fill="4" visible="no" active="yes"/>
 <layer number="121" name="_tsilk" color="7" fill="1" visible="no" active="yes"/>
@@
 <layer number="144" name="Drill_legend" color="7" fill="1" visible="no" active="yes"/>
 <layer number="151" name="HeatSink" color="7" fill="1" visible="no" active="yes"/>
+<layer number="199" name="Contour" color="7" fill="1" visible="yes" active="yes"/>
 <layer number="200" name="200bmp" color="1" fill="10" visible="no" active="yes"/>
 <layer number="201" name="201bmp" color="2" fill="10" visible="no" active="yes"/>
@@
 <wire x1="0" y1="101.6" x2="0" y2="0" width="0" layer="20"/>
 <text x="5.08" y="96.52" size="1.778" layer="51">Marky's House</text>
+<text x="8.89" y="8.89" size="1.778" layer="51">VOL OSC &amp; TUNING</text>
 </plain>
 <attributes>
@@
 <element name="C18" library="SparkFun-Passives" package="CPOL-RADIAL-10UF-25V" value="1uF" x="19.05" y="19.05" rot="R180"/>
 <element name="C16" library="SparkFun-Passives" package="CAP-PTH-SMALLEZ" value="22pF" x="24.13" y="38.1" rot="R270"/>
-<element name="R22" library="SparkFun-Passives" package="AXIAL-0.3EZ" value="10K" x="34.29" y="24.13"/>
-<element name="R21" library="SparkFun-Passives" package="AXIAL-0.3EZ" value="2.2K" x="34.29" y="26.67"/>
-<element name="R40" library="SparkFun-Passives" package="AXIAL-0.3EZ" value="10K" x="34.29" y="21.59"/>
-<element name="Q7" library="transistor" package="TO92" value="2N3904" x="36.83" y="46.99" rot="R90"/>
-<element name="Q6" library="transistor" package="TO92" value="2N3904" x="30.48" y="46.99" rot="R90"/>
-<element name="R16" library="SparkFun-Passives" package="AXIAL-0.3EZ" value="2.2K" x="34.29" y="19.05"/>
+<element name="R22" library="SparkFun-Passives" package="AXIAL-0.3EZ" value="10K" x="34.29" y="21.59"/>
+<element name="R21" library="SparkFun-Passives" package="AXIAL-0.3EZ" value="2.2K" x="34.29" y="24.13"/>
+<element name="R40" library="SparkFun-Passives" package="AXIAL-0.3EZ" value="10K" x="34.29" y="19.05"/>
+<element name="Q7" library="transistor" package="TO92" value="" x="36.83" y="46.99" rot="R90"/>
+<element name="Q6" library="transistor" package="TO92" value="" x="30.48" y="46.99" rot="R90"/>
+<element name="R16" library="SparkFun-Passives" package="AXIAL-0.3EZ" value="2.2K" x="34.29" y="16.51"/>
+<element name="C13" library="SparkFun-Capacitors" package="CPOL-RADIAL-1000UF-25V" value="22uF" x="22.86" y="58.42"/>
+<element name="C15" library="capacitor-wima" package="C5B3" value="6800pF" x="36" y="35.46" rot="R90"/>
+<element name="L11" library="marky-parts" package="SLOT-TEN" value="47uH" x="38.1" y="59.69"/>
+<element name="L14" library="marky-parts" package="FIXED-INDUCTOR-API-DELEVAN" value="22uH" x="44.45" y="38.1"/>
+<element name="C14" library="SparkFun-Capacitors" package="CAP-PTH-LARGE" value="1800pF" x="30.48" y="33.02" rot="R270"/>
+<element name="D3" library="diode" package="DO41-10" value="1N4004" x="60.96" y="73.66" rot="R90"/>
+<element name="U2" library="marky-parts" package="TO-92" value="LM79L12" x="72.7075" y="78.4225" rot="R180"/>
+<element name="U1" library="marky-parts" package="TO-92" value="LM78L12" x="73.3425" y="62.865"/>
+<element name="D1" library="diode" package="DO41-10" value="1N4004" x="70.1675" y="40.9575"/>
 </elements>
 <signals>
@@
 <contactref element="R21" pad="P$2"/>
 <wire x1="10.16" y1="19.05" x2="11.43" y2="33.02" width="0" layer="19" extent="1-1"/>
-<wire x1="38.1" y1="24.13" x2="10.16" y2="19.05" width="0" layer="19" extent="1-1"/>
-<wire x1="38.1" y1="26.67" x2="38.1" y2="24.13" width="0" layer="19" extent="1-1"/>
+<wire x1="38.1" y1="21.59" x2="10.16" y2="19.05" width="0" layer="19" extent="1-1"/>
+<wire x1="38.1" y1="24.13" x2="38.1" y2="21.59" width="0" layer="19" extent="1-1"/>
 </signal>
 <signal name="N$4">
 <contactref element="Q8" pad="1"/>
 <contactref element="C16" pad="1"/>
-<wire x1="24.13" y1="38.1" x2="16.51" y2="45.72" width="0" layer="19" extent="1-1"/>
+<contactref element="Q6" pad="1"/>
+<contactref element="L14" pad="P$2"/>
+<contactref element="C14" pad="1"/>
+<wire x1="24.13" y1="38.1" x2="30.48" y2="48.26" width="0" layer="19" extent="1-1"/>
+<wire x1="16.51" y1="45.72" x2="24.13" y2="38.1" width="0" layer="19" extent="1-1"/>
+<wire x1="44.45" y1="24.13" x2="24.13" y2="38.1" width="0" layer="19" extent="1-1"/>
+<wire x1="30.48" y1="37.846" x2="24.13" y2="38.1" width="0" layer="19" extent="1-1"/>
 </signal>
 <signal name="N$5">
@@
 <wire x1="20.32" y1="19.05" x2="19.05" y2="25.4" width="0" layer="19" extent="1-1"/>
 <wire x1="12.7" y1="19.05" x2="20.32" y2="19.05" width="0" layer="19" extent="1-1"/>
-<wire x1="38.1" y1="21.59" x2="12.7" y2="19.05" width="0" layer="19" extent="1-1"/>
+<wire x1="38.1" y1="19.05" x2="12.7" y2="19.05" width="0" layer="19" extent="1-1"/>
 </signal>
 <signal name="GND">
@@
 <contactref element="C18" pad="1"/>
 <contactref element="R15" pad="P$1"/>
-<wire x1="17.78" y1="19.05" x2="30.48" y2="26.67" width="0" layer="19" extent="1-1"/>
-<wire x1="11.43" y1="40.64" x2="17.78" y2="19.05" width="0" layer="19" extent="1-1"/>
+<contactref element="C13" pad="2"/>
+<contactref element="C15" pad="2"/>
+<contactref element="R17" pad="P$1"/>
+<contactref element="L11" pad="TAB@7"/>
+<contactref element="L11" pad="TAB@8"/>
+<contactref element="U2" pad="3"/>
+<contactref element="U1" pad="2"/>
+<wire x1="42.85" y1="59.69" x2="71.4375" y2="78.4225" width="0" layer="19" extent="1-1"/>
+<wire x1="33.35" y1="59.69" x2="42.85" y2="59.69" width="0" layer="19" extent="1-1"/>
+<wire x1="20.32" y1="58.42" x2="33.35" y2="59.69" width="0" layer="19" extent="1-1"/>
+<wire x1="11.43" y1="40.64" x2="20.32" y2="58.42" width="0" layer="19" extent="1-1"/>
+<wire x1="11.43" y1="36.83" x2="11.43" y2="40.64" width="0" layer="19" extent="1-1"/>
+<wire x1="17.78" y1="19.05" x2="11.43" y2="36.83" width="0" layer="19" extent="1-1"/>
+<wire x1="30.48" y1="24.13" x2="17.78" y2="19.05" width="0" layer="19" extent="1-1"/>
+<wire x1="36" y1="38" x2="30.48" y2="24.13" width="0" layer="19" extent="1-1"/>
+<wire x1="73.3425" y1="64.77" x2="17.78" y2="19.05" width="0" layer="19" extent="1-1"/>
 </signal>
 <signal name="N$7">
@@
 <contactref element="R40" pad="P$1"/>
 <contactref element="R16" pad="P$1"/>
-<wire x1="30.48" y1="21.59" x2="30.48" y2="24.13" width="0" layer="19" extent="1-1"/>
 <wire x1="30.48" y1="19.05" x2="30.48" y2="21.59" width="0" layer="19" extent="1-1"/>
+<wire x1="30.48" y1="16.51" x2="30.48" y2="19.05" width="0" layer="19" extent="1-1"/>
 </signal>
 <signal name="N$6">
@@
 <contactref element="R16" pad="P$2"/>
 <wire x1="36.83" y1="45.72" x2="30.48" y2="45.72" width="0" layer="19" extent="1-1"/>
-<wire x1="38.1" y1="19.05" x2="30.48" y2="45.72" width="0" layer="19" extent="1-1"/>
+<wire x1="38.1" y1="16.51" x2="30.48" y2="45.72" width="0" layer="19" extent="1-1"/>
 </signal>
 <signal name="N$8">
 <contactref element="Q6" pad="2"/>
+<contactref element="R15" pad="P$2"/>
+<wire x1="19.05" y1="40.64" x2="28.575" y2="46.99" width="0" layer="19" extent="1-1"/>
 </signal>
 <signal name="N$9">
 <contactref element="Q7" pad="2"/>
 <contactref element="R17" pad="P$2"/>
-<wire x1="19.05" y1="36.83" x2="34.925" y2="46.99" width="0" layer="19" extent="1-1"/>
+<contactref element="C15" pad="1"/>
+<contactref element="C14" pad="2"/>
+<wire x1="36" y1="32.92" x2="34.925" y2="46.99" width="0" layer="19" extent="1-1"/>
+<wire x1="19.05" y1="36.83" x2="36" y2="32.92" width="0" layer="19" extent="1-1"/>
+<wire x1="30.48" y1="28.448" x2="19.05" y2="36.83" width="0" layer="19" extent="1-1"/>
+</signal>
+<signal name="N$10">
+<contactref element="Q7" pad="1"/>
+<contactref element="C13" pad="1"/>
+<contactref element="L11" pad="IN$1"/>
+<wire x1="25.4" y1="58.42" x2="36.83" y2="48.26" width="0" layer="19" extent="1-1"/>
+<wire x1="34.6" y1="63.19" x2="25.4" y2="58.42" width="0" layer="19" extent="1-1"/>
+</signal>
+<signal name="N$11">
+<contactref element="L11" pad="OUT$3"/>
+<contactref element="L14" pad="P$1"/>
+<wire x1="44.45" y1="52.07" x2="41.6" y2="63.19" width="0" layer="19" extent="1-1"/>
+</signal>
+<signal name="N$12">
+<contactref element="U2" pad="2"/>
+<contactref element="D3" pad="A"/>
+<wire x1="72.7075" y1="76.5175" x2="60.96" y2="78.74" width="0" layer="19" extent="1-1"/>
+</signal>
+<signal name="N$13">
+<contactref element="D1" pad="C"/>
+<contactref element="U1" pad="1"/>
+<wire x1="72.0725" y1="62.865" x2="65.0875" y2="40.9575" width="0" layer="19" extent="1-1"/>
 </signal>
 </signals>
