File: eagle/Theremin/Theremin.sch (EAGLE design)
At the start: 98 parts, among them Q1 2N3904, Q2 2N3904, Q3 2N3904, Q4 2N3904, Q5 2N3904, Q6 2N3904, Q7 2N3904, Q8 2N3904, U1 LM78L12, U2 LM79L12

Commit message: Add headphone amp
various tweaks
Parts:
- removed AMP-SELECT: (no value), SparkFun-Connectors:M03LOCK_LONGPADS
- added C1-H: 0.1uF, SparkFun-Capacitors:CAPPTH
- added IC1-H: TL081, analog-devices:AD811N
- added JP7: HEADPHONE, SparkFun-Connectors:M03LOCK_LONGPADS
- added JP8: VOL TUNE, SparkFun-Connectors:M01PTH_LONGPAD
- added JP9: AMP-SELECT, SparkFun-Connectors:M03LOCK_LONGPADS
- added R1-H: 10K, SparkFun-Resistors:RESISTORPTH-1/4W
- added R2-H: 100K, SparkFun-Resistors:RESISTORPTH-1/4W
- added R3-H, R4-H: 330, SparkFun-Resistors:RESISTORPTH-1/4W
- D4, D5: value (none) -> 1N4148
- JP5: device SparkFun-Connectors:M01PTH_LONGPAD -> SparkFun-Connectors:M02LOCK_LONGPADS
Connections:
- new net N$31: C1-H.1, IC1-H.IN+, R1-H.2, R2-H.1
- new net N$55: C1-H.2, IC1-H.OUT, R2-H.2, R3-H.1, R4-H.1
- new net N$56: JP7.1, R3-H.2
- new net N$57: JP7.2, R4-H.2
- net 5V: now also IC1-H.+VS
- net GND: now also IC1-H.IN-, JP7.3
- net N$17: now also JP5.2
- net N$24: now also JP8.1
- net N$30: now also JP9.2; no longer AMP-SELECT.2
- net N$52: now also JP9.3; no longer AMP-SELECT.3
- net N$53: now also JP9.1; no longer AMP-SELECT.1
- net N$54: now also R1-H.1
- net VNEG: now also IC1-H.-VS

Commit message: Finalized board layout
Parts:
- added JP10, JP11, JP12: M02LOCK, SparkFun-Connectors:M02LOCK
- added U$1, U$2, U$3: (no value), marky-parts:GROUND-SCREW
- C1-H: value 0.1uF -> 100pF
- JP1: value (none) -> AUX
- JP2: device SparkFun-Connectors:M10LOCK_LONGPADS -> SparkFun-Connectors:M10"
- JP3: device SparkFun-Connectors:M02LOCK -> SparkFun-Connectors:M021X02_NO_SILK
- JP4: value VOL_ANT -> VOLUME_ANT; device SparkFun-Connectors:M02LOCK_LONGPADS -> SparkFun-Connectors:M021X02_NO_SILK
- JP5: device SparkFun-Connectors:M02LOCK_LONGPADS -> SparkFun-Connectors:M021X02_NO_SILK
- JP7: device SparkFun-Connectors:M03LOCK_LONGPADS -> SparkFun-Connectors:M031X03_NO_SILK
- JP9: device SparkFun-Connectors:M03LOCK_LONGPADS -> SparkFun-Connectors:M03LOCK
- U3: value (none) -> LM13700N
Connections:
- new net N$58: JP10.2, U$2.P$1
- new net N$59: JP11.2, U$1.P$1
- new net N$60: JP12.2, U$3.P$1
- net GND: now also JP10.1, JP11.1, JP12.1
Changed lines of the file:
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@@
 <setting verticaltext="up"/>
 </settings>
-<grid distance="0.1" unitdist="inch" unit="inch" style="lines" multiple="1" display="no" altdistance="0.01" altunitdist="inch" altunit="inch"/>
+<grid distance="0.05" unitdist="inch" unit="inch" style="lines" multiple="1" display="yes" altdistance="0.01" altunitdist="inch" altunit="inch"/>
 <layers>
 <layer number="1" name="Top" color="4" fill="1" visible="no" active="no"/>
@@
 <part name="C4" library="SparkFun-Passives" deviceset="CAP_POL" device="PTH2" value="1uF"/>
 <part name="C2" library="SparkFun-Capacitors" deviceset="CAP" device="PTH" value="15pF"/>
-<part name="U3" library="marky-parts" deviceset="LM13600" device=""/>
-<part name="JP1" library="SparkFun-Connectors" deviceset="M08" device="1X08"/>
+<part name="U3" library="marky-parts" deviceset="LM13600" device="" value="LM13700N"/>
+<part name="JP1" library="SparkFun-Connectors" deviceset="M08" device="1X08" value="AUX"/>
 <part name="GND12" library="supply1" deviceset="GND" device=""/>
 <part name="R38" library="SparkFun-Resistors" deviceset="RESISTOR" device="PTH-1/4W" value="47K"/>
@@
 <part name="R36" library="SparkFun-Resistors" deviceset="RESISTOR" device="PTH-1/4W" value="1M"/>
 <part name="R35" library="SparkFun-Resistors" deviceset="RESISTOR" device="PTH-1/4W" value="4.7M"/>
-<part name="JP2" library="SparkFun-Connectors" deviceset="M10" device="LOCK_LONGPADS" value="Front Panel"/>
+<part name="JP2" library="SparkFun-Connectors" deviceset="M10" device="&quot;" value="Front Panel"/>
 <part name="R30" library="SparkFun-Resistors" deviceset="RESISTOR" device="PTH-1/4W" value="47K"/>
 <part name="R29" library="SparkFun-Resistors" deviceset="RESISTOR" device="PTH-1/4W" value="100K"/>
@@
 <part name="P-5" library="SparkFun-Aesthetics" deviceset="VNEG" device="" value="-12V"/>
 <part name="SUPPLY4" library="SparkFun-Aesthetics" deviceset="5V" device="" value="12V"/>
-<part name="JP3" library="SparkFun-Connectors" deviceset="M02" device="LOCK" value="POWER IN"/>
+<part name="JP3" library="SparkFun-Connectors" deviceset="M02" device="1X02_NO_SILK" value="POWER IN"/>
 <part name="R27" library="SparkFun-Resistors" deviceset="RESISTOR" device="PTH-1/4W" value="150K"/>
 <part name="C6" library="SparkFun-Capacitors" deviceset="CAP" device="PTH" value="15pF"/>
@@
 <part name="P-8" library="SparkFun-Aesthetics" deviceset="VNEG" device="" value="-12V"/>
 <part name="C9" library="SparkFun-Capacitors" deviceset="CAP" device="PTH1" value="0.47uF"/>
-<part name="JP4" library="SparkFun-Connectors" deviceset="M02" device="LOCK_LONGPADS" value="VOL_ANT"/>
-<part name="JP5" library="SparkFun-Connectors" deviceset="M02" device="LOCK_LONGPADS" value="PITCH_ANT"/>
+<part name="JP4" library="SparkFun-Connectors" deviceset="M02" device="1X02_NO_SILK" value="VOLUME_ANT"/>
+<part name="JP5" library="SparkFun-Connectors" deviceset="M02" device="1X02_NO_SILK" value="PITCH_ANT"/>
 <part name="R14" library="SparkFun-Resistors" deviceset="RESISTOR" device="PTH-1/4W" value="1M"/>
 <part name="JP6" library="SparkFun-Connectors" deviceset="M02" device="LOCK" value="C28_SHORT"/>
 <part name="R33B" library="SparkFun-Resistors" deviceset="RESISTOR" device="PTH-1/4W" value="47K"/>
-<part name="JP9" library="SparkFun-Connectors" deviceset="M03" device="LOCK_LONGPADS" value="AMP-SELECT"/>
+<part name="JP9" library="SparkFun-Connectors" deviceset="M03" device="LOCK" value="AMP-SELECT"/>
 <part name="IC1-H" library="analog-devices" deviceset="AD811" device="N" value="TL081"/>
 <part name="P-9" library="SparkFun-Aesthetics" deviceset="VNEG" device="" value="-12V"/>
 <part name="SUPPLY7" library="SparkFun-Aesthetics" deviceset="5V" device="" value="12V"/>
-<part name="C1-H" library="SparkFun-Capacitors" deviceset="CAP" device="PTH" value="0.1uF"/>
+<part name="C1-H" library="SparkFun-Capacitors" deviceset="CAP" device="PTH" value="100pF"/>
 <part name="R1-H" library="SparkFun-Resistors" deviceset="RESISTOR" device="PTH-1/4W" value="10K"/>
 <part name="GND23" library="supply1" deviceset="GND" device=""/>
@@
 <part name="R3-H" library="SparkFun-Resistors" deviceset="RESISTOR" device="PTH-1/4W" value="330"/>
 <part name="R4-H" library="SparkFun-Resistors" deviceset="RESISTOR" device="PTH-1/4W" value="330"/>
-<part name="JP7" library="SparkFun-Connectors" deviceset="M03" device="LOCK_LONGPADS" value="HEADPHONE"/>
+<part name="JP7" library="SparkFun-Connectors" deviceset="M03" device="1X03_NO_SILK" value="HEADPHONE"/>
 <part name="GND24" library="supply1" deviceset="GND" device=""/>
 <part name="JP8" library="SparkFun-Connectors" deviceset="M01" device="PTH_LONGPAD" value="VOL TUNE"/>
+<part name="U$1" library="marky-parts" deviceset="GROUND-SCREW" device=""/>
+<part name="GND25" library="supply1" deviceset="GND" device=""/>
+<part name="U$2" library="marky-parts" deviceset="GROUND-SCREW" device=""/>
+<part name="U$3" library="marky-parts" deviceset="GROUND-SCREW" device=""/>
+<part name="JP10" library="SparkFun-Connectors" deviceset="M02" device="LOCK" value=""/>
+<part name="JP11" library="SparkFun-Connectors" deviceset="M02" device="LOCK" value=""/>
+<part name="JP12" library="SparkFun-Connectors" deviceset="M02" device="LOCK" value=""/>
+<part name="GND26" library="supply1" deviceset="GND" device=""/>
+<part name="GND27" library="supply1" deviceset="GND" device=""/>
 </parts>
 <sheets>
@@
 <instance part="GND24" gate="1" x="204.47" y="5.08"/>
 <instance part="JP8" gate="G$1" x="191.77" y="63.5" rot="R180"/>
+<instance part="U$1" gate="G$1" x="250.19" y="21.59"/>
+<instance part="GND25" gate="1" x="226.06" y="5.08"/>
+<instance part="U$2" gate="G$1" x="250.19" y="34.29"/>
+<instance part="U$3" gate="G$1" x="250.19" y="8.89"/>
+<instance part="JP10" gate="G$1" x="234.95" y="41.91" rot="R270"/>
+<instance part="JP11" gate="G$1" x="234.95" y="29.21" rot="R270"/>
+<instance part="JP12" gate="G$1" x="234.95" y="16.51" rot="R270"/>
+<instance part="GND26" gate="1" x="226.06" y="16.51"/>
+<instance part="GND27" gate="1" x="226.06" y="29.21"/>
 </instances>
 <busses>
@@
 <wire x1="204.47" y1="11.43" x2="208.28" y2="11.43" width="0.1524" layer="91"/>
 </segment>
+<segment>
+<pinref part="GND25" gate="1" pin="GND"/>
+<wire x1="226.06" y1="8.89" x2="226.06" y2="7.62" width="0.1524" layer="91"/>
+<pinref part="JP12" gate="G$1" pin="1"/>
+<wire x1="234.95" y1="8.89" x2="226.06" y2="8.89" width="0.1524" layer="91"/>
+</segment>
+<segment>
+<pinref part="JP10" gate="G$1" pin="1"/>
+<wire x1="234.95" y1="34.29" x2="226.06" y2="34.29" width="0.1524" layer="91"/>
+<pinref part="GND27" gate="1" pin="GND"/>
+<wire x1="226.06" y1="34.29" x2="226.06" y2="31.75" width="0.1524" layer="91"/>
+</segment>
+<segment>
+<pinref part="JP11" gate="G$1" pin="1"/>
+<wire x1="234.95" y1="21.59" x2="226.06" y2="21.59" width="0.1524" layer="91"/>
+<pinref part="GND26" gate="1" pin="GND"/>
+<wire x1="226.06" y1="21.59" x2="226.06" y2="19.05" width="0.1524" layer="91"/>
+</segment>
 </net>
 <net name="N$7" class="0">
@@
 <wire x1="222.25" y1="157.48" x2="222.25" y2="144.78" width="0.1524" layer="91"/>
 <wire x1="222.25" y1="144.78" x2="237.49" y2="144.78" width="0.1524" layer="91"/>
-<wire x1="237.49" y1="144.78" x2="237.49" y2="27.94" width="0.1524" layer="91"/>
+<wire x1="237.49" y1="144.78" x2="237.49" y2="48.26" width="0.1524" layer="91"/>
+<wire x1="237.49" y1="48.26" x2="195.58" y2="48.26" width="0.1524" layer="91"/>
+<wire x1="195.58" y1="48.26" x2="195.58" y2="27.94" width="0.1524" layer="91"/>
 <pinref part="JP2" gate="G$1" pin="6"/>
-<wire x1="237.49" y1="27.94" x2="100.33" y2="27.94" width="0.1524" layer="91"/>
+<wire x1="195.58" y1="27.94" x2="100.33" y2="27.94" width="0.1524" layer="91"/>
 <wire x1="100.33" y1="27.94" x2="100.33" y2="12.7" width="0.1524" layer="91"/>
 </segment>
@@
 <pinref part="JP2" gate="G$1" pin="5"/>
 <wire x1="102.87" y1="12.7" x2="102.87" y2="25.4" width="0.1524" layer="91"/>
-<wire x1="102.87" y1="25.4" x2="234.95" y2="25.4" width="0.1524" layer="91"/>
-<wire x1="234.95" y1="25.4" x2="234.95" y2="116.84" width="0.1524" layer="91"/>
+<wire x1="102.87" y1="25.4" x2="198.12" y2="25.4" width="0.1524" layer="91"/>
+<wire x1="198.12" y1="25.4" x2="198.12" y2="45.72" width="0.1524" layer="91"/>
+<wire x1="198.12" y1="45.72" x2="234.95" y2="45.72" width="0.1524" layer="91"/>
+<wire x1="234.95" y1="45.72" x2="234.95" y2="116.84" width="0.1524" layer="91"/>
 <wire x1="234.95" y1="116.84" x2="124.46" y2="116.84" width="0.1524" layer="91"/>
 <pinref part="R9" gate="G$1" pin="2"/>
@@
 </segment>
 </net>
+<net name="N$58" class="0">
+<segment>
+<pinref part="JP10" gate="G$1" pin="2"/>
+<pinref part="U$2" gate="G$1" pin="P$1"/>
+<wire x1="237.49" y1="34.29" x2="242.57" y2="34.29" width="0.1524" layer="91"/>
+</segment>
+</net>
+<net name="N$59" class="0">
+<segment>
+<pinref part="JP11" gate="G$1" pin="2"/>
+<pinref part="U$1" gate="G$1" pin="P$1"/>
+<wire x1="237.49" y1="21.59" x2="242.57" y2="21.59" width="0.1524" layer="91"/>
+</segment>
+</net>
+<net name="N$60" class="0">
+<segment>
+<pinref part="JP12" gate="G$1" pin="2"/>
+<pinref part="U$3" gate="G$1" pin="P$1"/>
+<wire x1="237.49" y1="8.89" x2="242.57" y2="8.89" width="0.1524" layer="91"/>
+</segment>
+</net>

Commit message: Theremin changes.
Other:
- note added: "LM78L12"
- note added: "LM79L12"
- note added: "U1"
- note added: "U2"
Changed lines of the file:
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@@
 <text x="118.11" y="168.91" size="1.778" layer="91">PITCH
 TUNING</text>
+<text x="40.64" y="40.64" size="1.778" layer="91" align="center">U1</text>
+<text x="40.64" y="7.62" size="1.778" layer="91" align="center">U2</text>
+<text x="40.64" y="44.45" size="1.778" layer="95" align="center">LM78L12</text>
+<text x="40.64" y="3.81" size="1.778" layer="95" align="center">LM79L12</text>
 </plain>
 <instances>
