File: eagle/UsbBoard/FTDI board.brd (EAGLE design)
At the start: 22.9 x 17.3 mm, 19 parts, among them U1 FT232RLSSOP, X1 USB-SMD-NS

Commit message: First shot at USB board
Parts:
- removed JP1: (no value), SparkFun:1X06-SMD-FEMALE-V2
- removed JP10, JP7, JP8, JP9: FIDUCIAL1X2, SparkFun:FIDUCIAL-1X2
- removed JP2: LOGO-SFESK, SparkFun:SFE-LOGO-FLAME
- removed U$2: LOGO-SFENW2, SparkFun:SFE-NEW-WEB
- added LED3: Green, SparkFun-LED:LED5MM
- added R3: 1K, SparkFun-Resistors:AXIAL-0.1
- C2: device SparkFun:0402-CAP -> SparkFun-Resistors:AXIAL-0.1
- LED1, LED2: device SparkFun:LED-0603 -> SparkFun-LED:LED5MM
- R1, R2: device SparkFun:0402-RES -> SparkFun-Resistors:AXIAL-0.1
- moved X1 46.7 mm to (25.4, 35.6)
- moved JP4 21.3 mm to (3.81, 12.7), turned to 90 degrees
- moved R2 17.1 mm to (25.4, 25.4), turned to 270 degrees
- moved SJ2 17.0 mm to (30.5, 16.3)
- moved JP3 16.1 mm to (36.8, 8.89)
- moved LED2 15.1 mm to (20.3, 25.4), turned to 180 degrees
- moved C2 11.8 mm to (15.2, 25.4), turned to 270 degrees
- moved LED1 10.6 mm to (10.2, 25.4), turned to 180 degrees
- moved R1 9.99 mm to (5.08, 25.4), turned to 270 degrees
- moved U1 8.64 mm to (15.2, 12.7)
- moved C1 5.68 mm to (10.2, 5.33)
- moved C5 5.09 mm to (15.2, 2.54)
Connections:
- new net N$3: LED3.A, R3.P$1
- net 5V: now also C2.P$1, R1.P$2, R2.P$2, R3.P$2; no longer C2.1, R1.2, R2.2
- net CTS: now also JP4.P$5; no longer JP1.2
- net DTR: now also JP4.P$1; no longer JP1.6
- net GND: now also C2.P$2, JP4.P$6, LED3.K; no longer C2.2, JP1.1
- net N$1: now also R1.P$1; no longer R1.1
- net N$2: now also R2.P$1; no longer R2.1
- net POWER: now also JP4.P$4; no longer JP1.3
- net RXI: now also JP4.P$3; no longer JP1.5
- net RXLED: now also LED2.K; no longer LED2.C
- net TXLED: now also LED1.K; no longer LED1.C
- net TXO: now also JP4.P$2; no longer JP1.4
Routing:
- net 5V: track 43.6 -> 0.00 mm, vias 1 -> 0
- net 3.3V: track 25.9 -> 0.00 mm, vias 1 -> 0
- net CTS: track 24.2 -> 0.00 mm, vias 1 -> 0
- net POWER: track 14.2 -> 0.00 mm, vias 1 -> 0
- net TXO: track 12.7 -> 0.00 mm, vias 1 -> 0
- net DTR: track 10.6 -> 0.00 mm, vias 1 -> 0
- net RXI: track 7.18 -> 0.00 mm, vias 1 -> 0
- net USB_D-: track 5.10 -> 0.00 mm
- net USB_D+: track 4.17 -> 0.00 mm
- net RXLED: track 3.55 -> 0.00 mm
- net TXLED: track 3.39 -> 0.00 mm
- net N$1: track 1.14 -> 0.00 mm
- net N$2: track 1.14 -> 0.00 mm
- removed copper zone on layer 16, net GND
Other:
- board outline removed
- board text removed: "3V3"
- board text removed: "BLK"
- board text removed: "CTS"
- board text removed: "DTR"
- board text removed: "GND"
- board text removed: "GRN"
- board text removed: "RXI"
- board text removed: "TXO"
