File: eagle/UsbBoard/FTDI board.sch (EAGLE design)
At the start: 19 parts, among them U1 FT232RLSSOP, X1 USB-SMD-NS

Commit message: First shot at USB board
Parts:
- removed JP1: (no value), SparkFun:M06SMD-FEMALE-V2
- removed JP10, JP7, JP8, JP9: FIDUCIAL1X2, SparkFun:FIDUCIAL1X2
- removed JP2: LOGO-SFESK, SparkFun:LOGO-SFESK
- removed U$2: LOGO-SFENW2, SparkFun:LOGO-SFENW2
- added LED3: Green, SparkFun-LED:LED5MM
- added R3: 1K, SparkFun-Resistors:RESISTORPTH-1/4W-VERT
- C2: device SparkFun:CAP0402-CAP -> SparkFun-Resistors:RESISTORPTH-1/4W-VERT
- LED1, LED2: device SparkFun:LED0603 -> SparkFun-LED:LED5MM
- R1, R2: device SparkFun:RESISTOR0402-RES -> SparkFun-Resistors:RESISTORPTH-1/4W-VERT
Connections:
- new net N$3: LED3.A, R3.1
- net 5V: now also R3.2
- net CTS: now also JP4.CTS; no longer JP1.2
- net DTR: now also JP4.DTR; no longer JP1.6
- net GND: now also JP4.GND, LED3.C; no longer JP1.1
- net POWER: now also JP4.VCC; no longer JP1.3
- net RXI: now also JP4.RXI; no longer JP1.5
- net TXO: now also JP4.TXO; no longer JP1.4
Other:
- moved on the sheet: JP4
Changed lines of the file:
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@@
 </classes>
 <parts>
-<part name="C2" library="SparkFun" deviceset="CAP" device="0402-CAP" value="0.1uF"/>
+<part name="C2" library="SparkFun-Resistors" deviceset="RESISTOR" device="PTH-1/4W-VERT" value="0.1uF"/>
 <part name="C5" library="SparkFun" deviceset="CAP_POL" device="1206" value="10uF"/>
 <part name="C1" library="SparkFun" deviceset="CAP" device="0402-CAP" value="0.1uF"/>
@@
 <part name="P+1" library="SparkFun" deviceset="VCC" device="" value="3.3V"/>
 <part name="FRAME1" library="SparkFun" deviceset="FRAME-LETTER" device=""/>
-<part name="U$2" library="SparkFun" deviceset="LOGO-SFE" device="NW2"/>
 <part name="U1" library="SparkFun" deviceset="FT232RL" device="SSOP"/>
 <part name="GND7" library="SparkFun" deviceset="GND" device=""/>
 <part name="GND8" library="SparkFun" deviceset="GND" device=""/>
-<part name="R1" library="SparkFun" deviceset="RESISTOR" device="0402-RES" value="1K"/>
-<part name="R2" library="SparkFun" deviceset="RESISTOR" device="0402-RES" value="1K"/>
-<part name="LED1" library="SparkFun" deviceset="LED" device="0603" value="Red"/>
-<part name="LED2" library="SparkFun" deviceset="LED" device="0603" value="Green"/>
+<part name="R1" library="SparkFun-Resistors" deviceset="RESISTOR" device="PTH-1/4W-VERT" value="1K"/>
+<part name="R2" library="SparkFun-Resistors" deviceset="RESISTOR" device="PTH-1/4W-VERT" value="1K"/>
+<part name="LED1" library="SparkFun-LED" deviceset="LED" device="5MM" value="Red"/>
+<part name="LED2" library="SparkFun-LED" deviceset="LED" device="5MM" value="Green"/>
 <part name="SJ2" library="SparkFun" deviceset="SOLDERJUMPER_2WAY" device="S"/>
 <part name="U$1" library="SparkFun" deviceset="5V" device=""/>
 <part name="U$3" library="SparkFun" deviceset="5V" device=""/>
 <part name="U$4" library="SparkFun" deviceset="5V" device=""/>
-<part name="JP2" library="SparkFun" deviceset="LOGO-SFE" device="SK"/>
-<part name="JP1" library="SparkFun" deviceset="M06" device="SMD-FEMALE-V2"/>
-<part name="JP7" library="SparkFun" deviceset="FIDUCIAL" device="1X2"/>
-<part name="JP8" library="SparkFun" deviceset="FIDUCIAL" device="1X2"/>
-<part name="JP9" library="SparkFun" deviceset="FIDUCIAL" device="1X2"/>
-<part name="JP10" library="SparkFun" deviceset="FIDUCIAL" device="1X2"/>
 <part name="JP3" library="SparkFun-Connectors" deviceset="M04" device="LOCK"/>
 <part name="X1" library="SparkFun" deviceset="USB" device="-SMD-NS"/>
 <part name="JP4" library="SparkFun-Connectors" deviceset="FTDI_DEVICE" device=""/>
+<part name="R3" library="SparkFun-Resistors" deviceset="RESISTOR" device="PTH-1/4W-VERT" value="1K"/>
+<part name="LED3" library="SparkFun-LED" deviceset="LED" device="5MM" value="Green"/>
+<part name="U$5" library="SparkFun" deviceset="5V" device=""/>
+<part name="GND3" library="SparkFun" deviceset="GND" device=""/>
 </parts>
 <sheets>
@@
 <instance part="FRAME1" gate="G$1" x="0" y="0"/>
 <instance part="FRAME1" gate="G$2" x="147.32" y="0"/>
-<instance part="U$2" gate="G$1" x="241.3" y="17.78"/>
 <instance part="U1" gate="G$1" x="124.46" y="109.22"/>
 <instance part="GND7" gate="1" x="66.04" y="101.6"/>
@@
 <instance part="U$3" gate="G$1" x="93.98" y="132.08"/>
 <instance part="U$4" gate="G$1" x="165.1" y="127"/>
-<instance part="JP2" gate="G$1" x="231.14" y="17.78"/>
-<instance part="JP1" gate="G$1" x="208.28" y="109.22" rot="R180"/>
-<instance part="JP7" gate="G$1" x="154.94" y="27.94"/>
-<instance part="JP8" gate="G$1" x="160.02" y="27.94"/>
-<instance part="JP9" gate="G$1" x="165.1" y="27.94"/>
-<instance part="JP10" gate="G$1" x="170.18" y="27.94"/>
 <instance part="JP3" gate="G$1" x="33.02" y="127"/>
 <instance part="X1" gate="G$1" x="20.32" y="124.46" rot="R180"/>
-<instance part="JP4" gate="G$1" x="226.06" y="109.22"/>
+<instance part="JP4" gate="G$1" x="210.82" y="111.76"/>
+<instance part="R3" gate="G$1" x="187.96" y="144.78" rot="R90"/>
+<instance part="LED3" gate="G$1" x="187.96" y="134.62"/>
+<instance part="U$5" gate="G$1" x="187.96" y="152.4"/>
+<instance part="GND3" gate="1" x="187.96" y="124.46"/>
 </instances>
 <busses>
@@
 </segment>
 <segment>
-<wire x1="66.04" y1="106.68" x2="66.04" y2="104.14" width="0.1524" layer="91"/>
+<wire x1="71.12" y1="109.22" x2="66.04" y2="104.14" width="0.1524" layer="91"/>
 <pinref part="C2" gate="G$1" pin="2"/>
 <pinref part="GND7" gate="1" pin="GND"/>
@@
 </segment>
 <segment>
-<wire x1="203.2" y1="114.3" x2="193.04" y2="114.3" width="0.1524" layer="91"/>
-<label x="193.04" y="114.3" size="1.778" layer="95"/>
-<pinref part="JP1" gate="G$1" pin="1"/>
+<wire x1="205.74" y1="104.14" x2="193.04" y2="104.14" width="0.1524" layer="91"/>
+<label x="193.04" y="104.14" size="1.778" layer="95"/>
+<pinref part="JP4" gate="G$1" pin="GND"/>
+</segment>
+<segment>
+<wire x1="187.96" y1="127" x2="187.96" y2="129.54" width="0.1524" layer="91"/>
+<pinref part="LED3" gate="G$1" pin="C"/>
+<pinref part="GND3" gate="1" pin="GND"/>
 </segment>
 </net>
@@
 </segment>
 <segment>
-<wire x1="203.2" y1="111.76" x2="193.04" y2="111.76" width="0.1524" layer="91"/>
-<label x="193.04" y="111.76" size="1.778" layer="95"/>
-<pinref part="JP1" gate="G$1" pin="2"/>
+<wire x1="205.74" y1="106.68" x2="193.04" y2="106.68" width="0.1524" layer="91"/>
+<label x="193.04" y="106.68" size="1.778" layer="95"/>
+<pinref part="JP4" gate="G$1" pin="CTS"/>
 </segment>
 </net>
@@
 </segment>
 <segment>
-<wire x1="203.2" y1="101.6" x2="193.04" y2="101.6" width="0.1524" layer="91"/>
-<label x="193.04" y="101.6" size="1.778" layer="95"/>
-<pinref part="JP1" gate="G$1" pin="6"/>
+<wire x1="205.74" y1="116.84" x2="193.04" y2="116.84" width="0.1524" layer="91"/>
+<label x="193.04" y="116.84" size="1.778" layer="95"/>
+<pinref part="JP4" gate="G$1" pin="DTR"/>
 </segment>
 </net>
@@
 </segment>
 <segment>
-<wire x1="203.2" y1="106.68" x2="193.04" y2="106.68" width="0.1524" layer="91"/>
-<label x="193.04" y="106.68" size="1.778" layer="95"/>
-<pinref part="JP1" gate="G$1" pin="4"/>
+<wire x1="205.74" y1="114.3" x2="193.04" y2="114.3" width="0.1524" layer="91"/>
+<label x="193.04" y="114.3" size="1.778" layer="95"/>
+<pinref part="JP4" gate="G$1" pin="TXO"/>
 </segment>
 </net>
@@
 </segment>
 <segment>
-<wire x1="203.2" y1="104.14" x2="193.04" y2="104.14" width="0.1524" layer="91"/>
-<label x="193.04" y="104.14" size="1.778" layer="95"/>
-<pinref part="JP1" gate="G$1" pin="5"/>
+<wire x1="205.74" y1="111.76" x2="193.04" y2="111.76" width="0.1524" layer="91"/>
+<label x="193.04" y="111.76" size="1.778" layer="95"/>
+<pinref part="JP4" gate="G$1" pin="RXI"/>
 </segment>
 </net>
@@
 </segment>
 <segment>
-<wire x1="203.2" y1="109.22" x2="190.5" y2="109.22" width="0.1524" layer="91"/>
+<wire x1="205.74" y1="109.22" x2="190.5" y2="109.22" width="0.1524" layer="91"/>
 <label x="193.04" y="109.22" size="1.778" layer="95"/>
 <pinref part="SJ2" gate="G$1" pin="2"/>
-<pinref part="JP1" gate="G$1" pin="3"/>
+<pinref part="JP4" gate="G$1" pin="VCC"/>
 </segment>
 </net>
@@
 <wire x1="93.98" y1="119.38" x2="109.22" y2="119.38" width="0.1524" layer="91"/>
 <wire x1="76.2" y1="114.3" x2="76.2" y2="129.54" width="0.1524" layer="91"/>
-<wire x1="66.04" y1="114.3" x2="66.04" y2="129.54" width="0.1524" layer="91"/>
+<wire x1="60.96" y1="109.22" x2="66.04" y2="129.54" width="0.1524" layer="91"/>
 <wire x1="38.1" y1="129.54" x2="66.04" y2="129.54" width="0.1524" layer="91"/>
 <wire x1="93.98" y1="132.08" x2="93.98" y2="129.54" width="0.1524" layer="91"/>
@@
 <pinref part="SJ2" gate="G$1" pin="1"/>
 </segment>
-</net>
+<segment>
+<wire x1="187.96" y1="152.4" x2="187.96" y2="149.86" width="0.1524" layer="91"/>
+<pinref part="R3" gate="G$1" pin="2"/>
+<pinref part="U$5" gate="G$1" pin="5V"/>
+</segment>
+</net>
+<net name="N$3" class="0">
+<segment>
+<wire x1="187.96" y1="139.7" x2="187.96" y2="137.16" width="0.1524" layer="91"/>
+<pinref part="R3" gate="G$1" pin="1"/>
+<pinref part="LED3" gate="G$1" pin="A"/>
+</segment>
+</net>
