File: eagle/UsbAtMega/UsbAtMega.sch (EAGLE design)
At the start: 16 parts, among them U1 ATMEGA328P_PDIP, U2 FT232RLSSOP

Commit message: tweaks
Parts:
- added JP1: (no value), SparkFun-Connectors:M06SIP
Connections:
- removed net 5V1: C5.1
- new net N$10: JP1.5, U1.PC4(ADC4/SDA)
- new net N$11: JP1.4, U1.PC3(ADC3)
- new net N$12: JP1.3, U1.PC2(ADC2)
- new net N$18: JP1.2, U1.PC1(ADC1)
- new net N$19: JP1.1, U1.PC0(ADC0)
- new net N$9: JP1.6, U1.PC5(ADC5/SCL)
- net 5V: now also C5.1
- net N$1: now also U1.PC6(/RESET)
- net N$7: now also U1.PB6(XTAL1/TOSC1)
- net N$8: now also U1.PB7(XTAL2/TOSC2)
Other:
- moved on the sheet: C5, Y1
Changed lines of the file:
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@@
 <part name="Y1" library="SparkFun-FreqCtrl" deviceset="RESONATOR" device="PTH"/>
 <part name="C5" library="SparkFun-Passives" deviceset="CAP" device="PTH" value="0.1uF"/>
+<part name="JP1" library="SparkFun-Connectors" deviceset="M06" device="SIP"/>
 </parts>
 <sheets>
@@
 <instance part="GND5" gate="1" x="144.78" y="106.68"/>
 <instance part="SUPPLY3" gate="G$1" x="119.38" y="190.5"/>
-<instance part="Y1" gate="G$1" x="147.32" y="142.24" rot="R270"/>
-<instance part="C5" gate="G$1" x="132.08" y="142.24"/>
+<instance part="Y1" gate="G$1" x="144.78" y="142.24" rot="R270"/>
+<instance part="C5" gate="G$1" x="132.08" y="139.7"/>
+<instance part="JP1" gate="G$1" x="210.82" y="165.1" rot="R180"/>
 </instances>
 <busses>
@@
 <junction x="144.78" y="114.3"/>
 <pinref part="C5" gate="G$1" pin="2"/>
-<wire x1="132.08" y1="114.3" x2="132.08" y2="139.7" width="0.1524" layer="91"/>
+<wire x1="132.08" y1="114.3" x2="132.08" y2="137.16" width="0.1524" layer="91"/>
 <wire x1="132.08" y1="114.3" x2="144.78" y2="114.3" width="0.1524" layer="91"/>
 </segment>
@@
 <pinref part="SUPPLY3" gate="G$1" pin="5V"/>
 <wire x1="149.86" y1="162.56" x2="142.24" y2="162.56" width="0.1524" layer="91"/>
-<wire x1="142.24" y1="162.56" x2="119.38" y2="162.56" width="0.1524" layer="91"/>
+<wire x1="142.24" y1="162.56" x2="132.08" y2="162.56" width="0.1524" layer="91"/>
+<wire x1="132.08" y1="162.56" x2="119.38" y2="162.56" width="0.1524" layer="91"/>
 <wire x1="119.38" y1="162.56" x2="119.38" y2="165.1" width="0.1524" layer="91"/>
 <pinref part="U1" gate="G$1" pin="AVCC"/>
@@
 <wire x1="142.24" y1="154.94" x2="142.24" y2="162.56" width="0.1524" layer="91"/>
 <junction x="142.24" y="162.56"/>
+<pinref part="C5" gate="G$1" pin="1"/>
+<wire x1="132.08" y1="162.56" x2="132.08" y2="144.78" width="0.1524" layer="91"/>
+<junction x="132.08" y="162.56"/>
 </segment>
 </net>
@@
 <wire x1="144.78" y1="170.18" x2="129.54" y2="170.18" width="0.1524" layer="91"/>
 <wire x1="129.54" y1="170.18" x2="129.54" y2="175.26" width="0.1524" layer="91"/>
+<pinref part="U1" gate="G$1" pin="PC6(/RESET)"/>
 </segment>
 </net>
@@
 <pinref part="U2" gate="G$1" pin="DTR"/>
 <wire x1="33.02" y1="144.78" x2="43.18" y2="144.78" width="0.1524" layer="91"/>
-<wire x1="43.18" y1="144.78" x2="43.18" y2="208.28" width="0.1524" layer="91"/>
+<wire x1="43.18" y1="144.78" x2="43.18" y2="205.74" width="0.1524" layer="91"/>
 <pinref part="C4" gate="G$1" pin="1"/>
-<wire x1="43.18" y1="208.28" x2="144.78" y2="208.28" width="0.1524" layer="91"/>
+<wire x1="43.18" y1="205.74" x2="144.78" y2="208.28" width="0.1524" layer="91"/>
 <wire x1="144.78" y1="208.28" x2="144.78" y2="182.88" width="0.1524" layer="91"/>
 </segment>
@@
 <wire x1="33.02" y1="157.48" x2="40.64" y2="157.48" width="0.1524" layer="91"/>
 <wire x1="40.64" y1="157.48" x2="40.64" y2="203.2" width="0.1524" layer="91"/>
-<wire x1="40.64" y1="203.2" x2="213.36" y2="203.2" width="0.1524" layer="91"/>
-<wire x1="213.36" y1="203.2" x2="213.36" y2="147.32" width="0.1524" layer="91"/>
+<wire x1="40.64" y1="203.2" x2="218.44" y2="203.2" width="0.1524" layer="91"/>
+<wire x1="218.44" y1="203.2" x2="218.44" y2="147.32" width="0.1524" layer="91"/>
 <pinref part="U1" gate="G$1" pin="PD0(RXD)"/>
-<wire x1="213.36" y1="147.32" x2="198.12" y2="147.32" width="0.1524" layer="91"/>
+<wire x1="218.44" y1="147.32" x2="198.12" y2="147.32" width="0.1524" layer="91"/>
 </segment>
 </net>
@@
 <wire x1="33.02" y1="154.94" x2="38.1" y2="154.94" width="0.1524" layer="91"/>
 <wire x1="38.1" y1="154.94" x2="38.1" y2="213.36" width="0.1524" layer="91"/>
-<wire x1="38.1" y1="213.36" x2="215.9" y2="213.36" width="0.1524" layer="91"/>
-<wire x1="215.9" y1="213.36" x2="215.9" y2="144.78" width="0.1524" layer="91"/>
+<wire x1="38.1" y1="213.36" x2="220.98" y2="213.36" width="0.1524" layer="91"/>
+<wire x1="220.98" y1="213.36" x2="220.98" y2="144.78" width="0.1524" layer="91"/>
 <pinref part="U1" gate="G$1" pin="PD1(TXD)"/>
-<wire x1="215.9" y1="144.78" x2="198.12" y2="144.78" width="0.1524" layer="91"/>
+<wire x1="220.98" y1="144.78" x2="198.12" y2="144.78" width="0.1524" layer="91"/>
 </segment>
 </net>
@@
 <segment>
 <pinref part="Y1" gate="G$1" pin="1"/>
-<wire x1="149.86" y1="144.78" x2="147.32" y2="144.78" width="0.1524" layer="91"/>
+<pinref part="U1" gate="G$1" pin="PB6(XTAL1/TOSC1)"/>
+<wire x1="149.86" y1="144.78" x2="144.78" y2="144.78" width="0.1524" layer="91"/>
 </segment>
 </net>
@@
 <segment>
 <pinref part="Y1" gate="G$1" pin="3"/>
-<wire x1="149.86" y1="139.7" x2="147.32" y2="139.7" width="0.1524" layer="91"/>
-</segment>
-</net>
-<net name="5V1" class="0">
-<segment>
-<pinref part="C5" gate="G$1" pin="1"/>
-<wire x1="132.08" y1="162.56" x2="132.08" y2="147.32" width="0.1524" layer="91"/>
-</segment>
-</net>
+<wire x1="149.86" y1="139.7" x2="144.78" y2="139.7" width="0.1524" layer="91"/>
+<pinref part="U1" gate="G$1" pin="PB7(XTAL2/TOSC2)"/>
+</segment>
+</net>
+<net name="N$9" class="0">
+<segment>
+<pinref part="U1" gate="G$1" pin="PC5(ADC5/SCL)"/>
+<pinref part="JP1" gate="G$1" pin="6"/>
+<wire x1="198.12" y1="157.48" x2="205.74" y2="157.48" width="0.1524" layer="91"/>
+</segment>
+</net>
+<net name="N$10" class="0">
+<segment>
+<pinref part="U1" gate="G$1" pin="PC4(ADC4/SDA)"/>
+<pinref part="JP1" gate="G$1" pin="5"/>
+<wire x1="198.12" y1="160.02" x2="205.74" y2="160.02" width="0.1524" layer="91"/>
+</segment>
+</net>
+<net name="N$11" class="0">
+<segment>
+<pinref part="U1" gate="G$1" pin="PC3(ADC3)"/>
+<pinref part="JP1" gate="G$1" pin="4"/>
+<wire x1="198.12" y1="162.56" x2="205.74" y2="162.56" width="0.1524" layer="91"/>
+</segment>
+</net>
+<net name="N$12" class="0">
+<segment>
+<pinref part="U1" gate="G$1" pin="PC2(ADC2)"/>
+<pinref part="JP1" gate="G$1" pin="3"/>
+<wire x1="198.12" y1="165.1" x2="205.74" y2="165.1" width="0.1524" layer="91"/>
+</segment>
+</net>
+<net name="N$18" class="0">
+<segment>
+<pinref part="U1" gate="G$1" pin="PC1(ADC1)"/>
+<pinref part="JP1" gate="G$1" pin="2"/>
+<wire x1="198.12" y1="167.64" x2="205.74" y2="167.64" width="0.1524" layer="91"/>
+</segment>
+</net>
+<net name="N$19" class="0">
+<segment>
+<pinref part="U1" gate="G$1" pin="PC0(ADC0)"/>
+<pinref part="JP1" gate="G$1" pin="1"/>
+<wire x1="198.12" y1="170.18" x2="205.74" y2="170.18" width="0.1524" layer="91"/>
+</segment>
+</net>
